Commit message: 修复了一个会在ros2_control上出现的bug

File: urdf/body/robot_body.xacro (robot description, xacro)
@@ -12,5 +12,5 @@
     <xacro:body_link_with_sc name="left_wheel_link" body_kinematics_link="${body_kinematics_link}"
       body_inertials="${body_inertials}" />
-    <joint name="left_wheel_joint" type="continuous">
+    <joint name="${body_prefix}left_wheel_joint" type="continuous">
       <xacro:body_kinematics name="left_wheel_link" config="${body_kinematics}" />
       <parent link="${body_prefix}base_link" />
@@ -22,5 +22,5 @@
     <xacro:body_link_with_sc name="right_wheel_link" body_kinematics_link="${body_kinematics_link}"
       body_inertials="${body_inertials}" />
-    <joint name="right_wheel_joint" type="continuous">
+    <joint name="${body_prefix}right_wheel_joint" type="continuous">
       <xacro:body_kinematics name="right_wheel_link" config="${body_kinematics}" />
       <parent link="${body_prefix}base_link" />
